Commit message: The 1st success with jackal (os1-64 lidar)

File: Shared_folder/jackal_description/urdf/jackal.urdf.xacro (robot description, xacro)
@@ -177,5 +177,5 @@
        always points to the "active" IMU. When an upgrade IMU is connected, the
        internal_imu_link should remain, but imu_link should point to the upgrade one. -->
-  <!--link name="imu_link">
+  <link name="imu_link">
     <inertial>
       <mass value="0.001"/>
@@ -187,5 +187,5 @@
     <parent link="chassis_link" />
     <child link="imu_link" />
-  </joint-->
+  </joint>
   <!-- TODO: Same note as applies to imu_link -->
   <link name="navsat_link">

File: Shared_folder/jackal_description/urdf/jackal_3d.urdf (robot description, URDF)
Before this commit: robot jackal, 5 links, 4 joints
Links:
- removed link os_sensor
- added link os1_lidar
Joints:
- joint os_sensor_joint: child os_sensor -> os1_lidar; origin xyz=0 0 0.402 rpy=0 0 0 -> xyz=0 0 0.438 rpy=0 0 0

File: Shared_folder/jackal_description/urdf/roas.urdf.xacro (robot description, xacro)
@@ -38,6 +38,13 @@
     <origin xyz="0.180 0 0.295" rpy="0 0 0"/>
   </xacro:sensor_d435>
+<!--
   <xacro:sensor_os1 parent="base_link" name="os_sensor">
     <origin xyz="0 0 0.402" rpy="0 0 0"/>
   </xacro:sensor_os1>
+-->
+  <!-- OUSTER OS1-64 : added by jschoi-->
+  <xacro:include filename="$(find ouster_description)/urdf/OS1-64.urdf.xacro"/>
+  <xacro:OS1-64 parent="base_link" name="os1_sensor" hz="10" samples="220">
+    <origin xyz="0 0 0.438" rpy="0 0 0" />
+  </xacro:OS1-64>
 </robot>
